File: Electronics/FreeEEG.kicad_pcb (KiCad board)
At the start: 2 copper layers, 0 parts

Commit message: Starting final firmware development
Parts:
- added BT1: 9V, Connector_PinHeader_2.54mm:PinHeader_1x02_P2.54mm_Vertical, F.Cu at (124.0, 99.5)
- added C1: 10u, Capacitor_SMD:C_0805_2012Metric, F.Cu at (155.1, 89.0)
- added C10: 4.7n, Capacitor_SMD:C_0603_1608Metric, F.Cu at (165.9, 140.7)
- added C11: 4.7n, Capacitor_SMD:C_0603_1608Metric, F.Cu at (161.4, 140.7)
- added C12: 4.7n, Capacitor_SMD:C_0603_1608Metric, F.Cu at (159.8, 140.7)
- added C13: 4.7n, Capacitor_SMD:C_0603_1608Metric, F.Cu at (155.3, 140.7)
- added C14: 4.7n, Capacitor_SMD:C_0603_1608Metric, F.Cu at (153.8, 140.7)
- added C15: 4.7n, Capacitor_SMD:C_0603_1608Metric, F.Cu at (149.3, 140.7)
- added C16: 4.7n, Capacitor_SMD:C_0603_1608Metric, F.Cu at (147.8, 140.7)
- added C17: 4.7n, Capacitor_SMD:C_0603_1608Metric, F.Cu at (143.3, 140.7)
- added C18: 4.7n, Capacitor_SMD:C_0603_1608Metric, F.Cu at (141.8, 140.7)
- added C19: 4.7n, Capacitor_SMD:C_0603_1608Metric, F.Cu at (137.2, 140.7)
- added C2: 10n, Capacitor_SMD:C_0805_2012Metric, F.Cu at (150.9, 89.0)
- added C20: 4.7n, Capacitor_SMD:C_0603_1608Metric, F.Cu at (135.7, 140.7)
- added C21: 4.7n, Capacitor_SMD:C_0603_1608Metric, F.Cu at (131.2, 140.7)
- added C22: 4.7n, Capacitor_SMD:C_0603_1608Metric, F.Cu at (129.7, 140.7)
- added C23: 4.7n, Capacitor_SMD:C_0603_1608Metric, F.Cu at (125.2, 140.7)
- added C24: 4.7n, Capacitor_SMD:C_0603_1608Metric, F.Cu at (174.9, 140.8)
- added C25: 1u, Capacitor_SMD:C_0805_2012Metric, F.Cu at (165.3, 126.6)
- added C26: 1u, Capacitor_SMD:C_0805_2012Metric, F.Cu at (173.6, 126.8)
- added C27: 1u, Capacitor_SMD:C_0805_2012Metric, F.Cu at (151.7, 85.0)
- added C28: 33u, Capacitor_SMD:C_1206_3216Metric, F.Cu at (126.9, 128.0)
- added C29: 33u, Capacitor_SMD:C_1206_3216Metric, F.Cu at (132.3, 117.9)
- added C3: 1u, Capacitor_SMD:C_0805_2012Metric, F.Cu at (155.9, 79.1)
- added C30: 10n, Capacitor_SMD:C_0603_1608Metric, F.Cu at (138.9, 133.3)
- added C31: 10u, Capacitor_SMD:C_0805_2012Metric, F.Cu at (161.5, 128.5)
- added C32: 0.1u, Capacitor_SMD:C_0603_1608Metric, F.Cu at (161.5, 126.6)
- added C33: 100u, Capacitor_SMD:C_Elec_6.3x7.7, F.Cu at (160.6, 121.4)
- added C34: 1u, Capacitor_SMD:C_0603_1608Metric, F.Cu at (155.0, 121.5)
- added C35: 1u, Capacitor_SMD:C_0603_1608Metric, F.Cu at (138.8, 124.6)
- added C36: 0.1u, Capacitor_SMD:C_0603_1608Metric, F.Cu at (138.8, 126.1)
- added C37: 1u, Capacitor_SMD:C_0603_1608Metric, F.Cu at (158.2, 126.3)
- added C38: 1u, Capacitor_SMD:C_0603_1608Metric, F.Cu at (140.5, 121.7)
- added C39: 0.1u, Capacitor_SMD:C_0603_1608Metric, F.Cu at (142.0, 121.7)
- added C4: 100n, Capacitor_SMD:C_0805_2012Metric, F.Cu at (155.9, 77.0)
- added C40: 1u, Capacitor_SMD:C_0603_1608Metric, F.Cu at (158.2, 128.2)
- added C41: 0.1u, Capacitor_SMD:C_0603_1608Metric, F.Cu at (158.2, 129.7)
- added C42: 1u, Capacitor_SMD:C_0603_1608Metric, F.Cu at (138.8, 127.7)
- added C43: 0.1u, Capacitor_SMD:C_0603_1608Metric, F.Cu at (138.8, 129.2)
- added C44: 1u, Capacitor_SMD:C_0603_1608Metric, F.Cu at (137.8, 121.5)
- added C45: 0.1u, Capacitor_SMD:C_0603_1608Metric, F.Cu at (137.8, 123.0)
- added C46: 10n, Capacitor_SMD:C_0603_1608Metric, F.Cu at (170.3, 116.9)
- added C47: 100n, Capacitor_SMD:C_0603_1608Metric, F.Cu at (172.3, 117.5)
- added C48: 2.2n, Capacitor_SMD:C_0603_1608Metric, F.Cu at (173.3, 109.0)
- added C5: 10u, Capacitor_SMD:C_0805_2012Metric, F.Cu at (153.0, 89.0)
- added C6: 330u, Capacitor_SMD:C_Elec_8x10.2, F.Cu at (127.5, 76.5)
- added C7: 470u, Capacitor_SMD:C_Elec_8x10.2, F.Cu at (139.6, 91.7)
- added C8: 4.7n, Capacitor_SMD:C_0603_1608Metric, F.Cu at (171.9, 140.8)
- added C9: 4.7n, Capacitor_SMD:C_0603_1608Metric, F.Cu at (167.4, 140.7)
- added D1: ON_LED, LED_SMD:LED_0805_2012Metric, F.Cu at (128.3, 96.0)
- added D2: SS54B, Diode_SMD:D_SMB, F.Cu at (131.5, 86.7)
- added D3: LED_RAGB, XL-3528RGBW-HM:XL-3528RGBW-HM, F.Cu at (129.7, 111.0)
- added J1: ConnElectrodes, Connector_PinHeader_2.54mm:PinHeader_2x10_P2.54mm_Vertical, F.Cu at (140.3, 152.0)
- added J2: 10137065-00021LF, 10137065-00021LF:AMPHENOL_10137065-00021LF, F.Cu at (150.0, 65.9)
- added L1: 47u, Inductor_SMD:L_Bourns_SRP7028A_7.3x6.6mm, F.Cu at (139.3, 80.4)
- added MICRO_SD1: TF-01A, TF-01A:TF-01A, F.Cu at (168.0, 71.5)
- added Q1: 2N7002, Package_TO_SOT_SMD:SOT-23, F.Cu at (137.0, 104.1)
- added Q2: 2N7002, Package_TO_SOT_SMD:SOT-23, F.Cu at (133.5, 104.1)
- added Q3: 2N7002, Package_TO_SOT_SMD:SOT-23, F.Cu at (140.6, 103.9)
- added R1: 10k, Resistor_SMD:R_0603_1608Metric, F.Cu at (160.0, 82.6)
- added R10: 33k, Resistor_SMD:R_0603_1608Metric, F.Cu at (145.6, 118.5)
- added R11: 33k, Resistor_SMD:R_0603_1608Metric, F.Cu at (144.1, 118.5)
- added R12: 10k, Resistor_SMD:R_0603_1608Metric, F.Cu at (155.3, 115.1)
- added R13: 10k, Resistor_SMD:R_0603_1608Metric, F.Cu at (153.8, 115.1)
- added R14: 400, Resistor_SMD:R_0805_2012Metric, F.Cu at (131.9, 96.0)
- added R15: 4.99k, Resistor_SMD:R_0603_1608Metric, F.Cu at (168.9, 140.7)
- added R16: 4.99k, Resistor_SMD:R_0603_1608Metric, F.Cu at (170.4, 140.7)
- added R17: 4.99k, Resistor_SMD:R_0603_1608Metric, F.Cu at (164.4, 140.7)
- added R18: 4.99k, Resistor_SMD:R_0603_1608Metric, F.Cu at (162.9, 140.7)
- added R19: 4.99k, Resistor_SMD:R_0603_1608Metric, F.Cu at (158.3, 140.7)
- added R2: 10k, Resistor_SMD:R_0603_1608Metric, F.Cu at (160.0, 81.1)
- added R20: 4.99k, Resistor_SMD:R_0603_1608Metric, F.Cu at (156.8, 140.7)
- added R21: 4.99k, Resistor_SMD:R_0603_1608Metric, F.Cu at (152.3, 140.7)
- added R22: 4.99k, Resistor_SMD:R_0603_1608Metric, F.Cu at (150.8, 140.7)
- added R23: 4.99k, Resistor_SMD:R_0603_1608Metric, F.Cu at (146.3, 140.7)
- added R24: 4.99k, Resistor_SMD:R_0603_1608Metric, F.Cu at (144.8, 140.7)
- added R25: 4.99k, Resistor_SMD:R_0603_1608Metric, F.Cu at (140.2, 140.7)
- added R26: 4.99k, Resistor_SMD:R_0603_1608Metric, F.Cu at (138.7, 140.7)
- added R27: 4.99k, Resistor_SMD:R_0603_1608Metric, F.Cu at (134.2, 140.7)
- added R28: 4.99k, Resistor_SMD:R_0603_1608Metric, F.Cu at (132.7, 140.7)
- added R29: 4.99k, Resistor_SMD:R_0603_1608Metric, F.Cu at (128.2, 140.7)
- added R3: 10k, Resistor_SMD:R_0603_1608Metric, F.Cu at (172.3, 82.3)
- added R30: 4.99k, Resistor_SMD:R_0603_1608Metric, F.Cu at (126.7, 140.7)
- added R31: 4.99k, Resistor_SMD:R_0603_1608Metric, F.Cu at (173.4, 140.8)
- added R32: 2M, Resistor_SMD:R_0603_1608Metric, F.Cu at (173.5, 122.8)
- added R33: 2M, Resistor_SMD:R_0603_1608Metric, F.Cu at (173.5, 124.8)
- added R34: 33k, Resistor_SMD:R_0603_1608Metric, F.Cu at (135.2, 69.6)
- added R35: 10k, Resistor_SMD:R_0603_1608Metric, F.Cu at (153.8, 85.0)
- added R36: 392k, Resistor_SMD:R_0603_1608Metric, F.Cu at (138.9, 131.3)
- added R37: 2M, Resistor_SMD:R_0603_1608Metric, F.Cu at (128.8, 102.7)
- added R38: 1M, Resistor_SMD:R_0603_1608Metric, F.Cu at (128.8, 104.3)
- added R39: 720, Resistor_SMD:R_0805_2012Metric, F.Cu at (134.8, 112.3)
- added R4: 10k, Resistor_SMD:R_0603_1608Metric, F.Cu at (172.3, 83.8)
- added R40: 610, Resistor_SMD:R_0805_2012Metric, F.Cu at (134.8, 110.2)
- added R41: 610, Resistor_SMD:R_0805_2012Metric, F.Cu at (134.8, 114.3)
- added R42: 10, Resistor_SMD:R_0603_1608Metric, F.Cu at (134.5, 99.8)
- added R43: 10, Resistor_SMD:R_0603_1608Metric, F.Cu at (141.5, 100.0)
- added R44: 10, Resistor_SMD:R_0603_1608Metric, F.Cu at (138.0, 99.8)
- added R45: 10k, Resistor_SMD:R_0603_1608Metric, F.Cu at (152.3, 115.1)
- added R46: 4.99k, Resistor_SMD:R_0603_1608Metric, F.Cu at (176.8, 140.8)
- added R5: 10k, Resistor_SMD:R_0603_1608Metric, F.Cu at (160.0, 84.1)
- added R6: 5.1k, Resistor_SMD:R_0603_1608Metric, F.Cu at (146.8, 74.8)
- added R7: 5.1k, Resistor_SMD:R_0603_1608Metric, F.Cu at (151.5, 74.1)
- added R8: 33k, Resistor_SMD:R_0603_1608Metric, F.Cu at (149.3, 118.5)
- added R9: 33k, Resistor_SMD:R_0603_1608Metric, F.Cu at (147.1, 118.5)
- added SW1: ON_SW, K3-1260D-L1:K3-1260D-L1, F.Cu at (124.0, 106.5)
- added SW2: SEL_SW, K3-1260D-L1:K3-1260D-L1, F.Cu at (135.2, 66.0)
- added SW3: RST_BTN, K2-1187SQ-A4SW-06:K2-1187SQ-A4SW-06, F.Cu at (147.8, 82.8)
- added SW4: BOOT_BTN, K2-1187SQ-A4SW-06:K2-1187SQ-A4SW-06, F.Cu at (162.4, 110.5)
- added TP1: REF_TEST, TestPoint:TestPoint_Pad_D1.5mm, F.Cu at (161.5, 131.6)
- added TP2: GND_TEST, TestPoint:TestPoint_Pad_D1.5mm, F.Cu at (168.6, 121.4)
- added TP3: 3V3_TEST, TestPoint:TestPoint_Pad_D1.5mm, F.Cu at (127.2, 67.2)
- added U1: ADS1299, Package_QFP:TQFP-64_10x10mm_P0.5mm, F.Cu at (148.7, 127.8)
- added U2: OPA376xxDBV, Package_TO_SOT_SMD:SOT-23-5, F.Cu at (173.5, 130.4)
- added U3: ESP32-S3-WROOM-1, RF_Module:ESP32-S3-WROOM-1, F.Cu at (171.1, 94.8)
- added U4: OPA376xxDBV, Package_TO_SOT_SMD:SOT-23-5, F.Cu at (165.3, 130.2)
- added U5: XL1509-3.3, Package_SO:SOIC-8_3.9x4.9mm_P1.27mm, F.Cu at (126.4, 88.0)
- added U6: NCP1117-5.0_SOT223, Package_TO_SOT_SMD:SOT-223-3_TabPin2, F.Cu at (128.8, 122.8)
- added U7: MPU-6050, Sensor_Motion:InvenSense_QFN-24_4x4mm_P0.5mm, F.Cu at (171.7, 112.7)
Routing:
- net +3.3V: track 0.00 -> 241.2 mm, vias 0 -> 9
- net +5V: track 0.00 -> 83.3 mm
- net GND: track 0.00 -> 70.9 mm, vias 0 -> 75
- net BATT: track 0.00 -> 70.0 mm
- net RESET: track 0.00 -> 54.2 mm, vias 0 -> 2
- net BAT_MON: track 0.00 -> 54.1 mm, vias 0 -> 2
- net AFE_NDRDY: track 0.00 -> 52.9 mm, vias 0 -> 2
- net SEL: track 0.00 -> 50.1 mm, vias 0 -> 2
- net AFE_NCS: track 0.00 -> 38.8 mm, vias 0 -> 2
- net AFE_DOUT: track 0.00 -> 35.0 mm, vias 0 -> 2
- net AFE_START: track 0.00 -> 34.7 mm, vias 0 -> 2
- net LED_R: track 0.00 -> 34.4 mm, vias 0 -> 2
- net AFE_DIN: track 0.00 -> 34.3 mm, vias 0 -> 2
- net AFE_SCLK: track 0.00 -> 32.4 mm
- net SD_DAT0: track 0.00 -> 32.2 mm
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- added copper zone on B.Cu, net GND
- added copper zone on F.Cu, net GND
Other:
- board outline added: 56.3 x 91.6 mm
