File: Electronics/interface.kicad_sch (KiCad schematic)
At the start: 19 parts, among them J1 ConnElectrodes, J5 B2B-PH-SM4-TBT_LF, J6 ExtTrig, SW1 ON_SW, SW2 SEL_SW, SW3 RST_BTN

Commit message: [Electronics] version 1.0.0 of the PCB released.\n [Firmware] Added ICS43434 drivers and prepared code for reestructuration
Parts:
- removed J5: B2B-PH-SM4-TBT_LF, B2B-PH-SM4-TBT_LF__SN_:B2BPHSM4TBTLFSN, symbol B2B-PH-SM4-TBT_LF__SN_:B2B-PH-SM4-TBT_LF__SN_
- added J3: Conn_I2C, Connector_JST:JST_SH_SM04B-SRSS-TB_1x04-1MP_P1.00mm_Horizontal, symbol Connector_Generic_MountingPin:Conn_01x04_MountingPin
- added J4: battery_conn, Connector_Molex:Molex_PicoBlade_53261-0371_1x03-1MP_P1.25mm_Horizontal, symbol Connector_Generic_MountingPin:Conn_01x03_MountingPin
Connections:
- net +3.3V: now also J3.2 (Pin_2)
- net +BATT: now also J4.1 (Pin_1)
- net GND: now also J3.1 (Pin_1), J3.MP (MountPin), J4.3 (Pin_3), J4.MP (MountPin)
- new net I2C_SCL: J3.4 (Pin_4)
- new net I2C_SDA: J3.3 (Pin_3)
- no-connect marks 3 -> 2
Other:
- note added: "QWIIC interface"
- moved on the sheet: C27, R35, SW3
